Commit message: Update WSG-50 gripper and FTS sensor models

File: src/lwa4p_description/urdf/lwa4p.urdf.xacro (robot description, xacro)
@@ -89,17 +89,24 @@
                    xyz="0 0 0" rpy="-1.5708 0 0" effort="19" lower="${-lim}" upper="${lim}"/>
   <xacro:arm_link name="arm_6_link" stl="arm_6_link" material="schunk_grey"/>
-  <!-- tool flange face (end of the arm_6 mesh, z = 0.084) -->
+  <!-- Tool flange matching original Schunk schunk_lwa4p.urdf.xacro -->
   <joint name="arm_tool0_joint" type="fixed">
     <parent link="arm_6_link"/>
     <child link="arm_tool0"/>
-    <origin xyz="0 0 0.084" rpy="0 0 0"/>
+    <origin xyz="0 0 0.0751" rpy="0 0 3.14159"/>
   </joint>
   <link name="arm_tool0"/>
+  <!-- FTS-LWA Sensor -->
+  <xacro:include filename="$(find lwa4p_description)/urdf/fts_lwa.urdf.xacro"/>
+  <xacro:fts_lwa parent="arm_tool0" has_parent="true" tool_point="fts_lwa_tool_link">
+    <origin xyz="0 0 0" rpy="0 0 0"/>
+  </xacro:fts_lwa>
+  <!-- WSG-50 Gripper -->
   <xacro:arg name="gripper" default="true"/>
-  <!-- rotate the gripper about the flange axis if RViz doesn't match the real arm -->
   <xacro:arg name="gripper_yaw" default="1.5708"/>
   <xacro:if value="$(arg gripper)">
     <xacro:include filename="$(find lwa4p_description)/urdf/wsg50.urdf.xacro"/>
-    <xacro:wsg50 parent="arm_tool0" yaw="$(arg gripper_yaw)"/>
+    <xacro:wsg_50_xacro name="gripper" parent="fts_lwa_tool_link" tool_point="gripper_tcp">
+      <origin xyz="0 0 0" rpy="0 0 $(arg gripper_yaw)"/>
+    </xacro:wsg_50_xacro>
   </xacro:if>
 </robot>

File: src/lwa4p_description/urdf/wsg50.urdf.xacro (robot description, xacro)
@@ -1,87 +1,66 @@
 <?xml version="1.0"?>
-<!-- Weiss/Schunk WSG 50-110 on an adapter plate, simple box geometry.
-     From the WSG 50 manual (05.00, 389474, "3.1 Outer dimensions"):
-       housing 146 x 50 x 72.5 mm (x = jaw direction), Ø50 ISO mounting in the
-       centre of the bottom face, base jaws stick out to 96.5 mm (24 mm above
-       the housing), ~18 mm wide in x, jaw inner faces 0..110 mm apart.
-       Weight 1.15 kg, 5..80 N, 5..420 mm/s.
-     Measured on the real gripper: the mounted fingers reach 9.75 mm further
-       inwards than each jaw (fingertip gap = jaw width - 19.5 mm).
-     NOT measured yet (change when you know them):
-       adapter_h (flange -> housing bottom), jaw_d (jaw depth in y),
-       finger_t / finger_w / finger_l (finger thickness, width, length above
-       the jaw). finger_l is chosen so the fingertips are 162 mm above the
-       housing bottom, as in the earlier model (keeps gripper_tcp unchanged).
-     gripper_joint = fingertip GAP in metres (same number the gripper node,
-     MoveIt and `arm_cmd.sh grip` use). Each finger mimics half of it. -->
 <robot xmlns:xacro="http://www.ros.org/wiki/xacro">
-  <xacro:macro name="wsg50" params="parent yaw:=0">
-    <xacro:property name="adapter_h" value="0.020"/>
-    <xacro:property name="body_x" value="0.146"/>
-    <xacro:property name="body_y" value="0.050"/>
-    <xacro:property name="body_h" value="0.0725"/>
-    <xacro:property name="jaw_w" value="0.018"/>
-    <xacro:property name="jaw_d" value="0.030"/>
-    <xacro:property name="jaw_h" value="0.024"/>
-    <xacro:property name="jaw_inset" value="0.00975"/>
-    <xacro:property name="finger_t" value="0.020"/>
-    <xacro:property name="finger_w" value="0.030"/>
-    <xacro:property name="finger_l" value="0.0655"/>
-    <xacro:property name="gap_max" value="0.0895"/>
-    <material name="wsg_grey"><color rgba="0.6 0.6 0.62 1.0"/></material>
-    <material name="wsg_jaw"><color rgba="0.35 0.35 0.38 1.0"/></material>
-    <material name="wsg_black"><color rgba="0.1 0.1 0.1 1.0"/></material>
-    <joint name="gripper_adapter_joint" type="fixed">
+  <xacro:macro name="wsg_50_xacro" params="name parent *origin tool_point">
+    <!-- Connector plate from original Schunk assembly -->
+    <joint name="${name}_connector_gripper_joint" type="fixed">
+      <xacro:insert_block name="origin"/>
       <parent link="${parent}"/>
-      <child link="gripper_adapter_link"/>
-      <origin xyz="0 0 0" rpy="0 0 ${yaw}"/>
+      <child link="${name}_connector_link"/>
     </joint>
-    <link name="gripper_adapter_link">
+    <link name="${name}_connector_link">
+      <inertial>
+        <mass value="0.01"/>
+        <origin xyz="0 0 0"/>
+        <inertia ixx="0.001" ixy="0.0" ixz="0.0" iyy="0.001" iyz="0.0" izz="0.001"/>
+      </inertial>
       <visual>
-        <origin xyz="0 0 ${adapter_h / 2}"/>
-        <geometry><cylinder radius="0.0325" length="${adapter_h}"/></geometry>
-        <material name="wsg_grey"/>
+        <origin rpy="0 0 0" xyz="0 0 0.007"/>
+        <geometry>
+          <cylinder length="0.014" radius="0.030"/>
+        </geometry>
+        <material name="schunk_grey"/>
       </visual>
       <collision>
-        <origin xyz="0 0 ${adapter_h / 2}"/>
-        <geometry><cylinder radius="0.0325" length="${adapter_h}"/></geometry>
+        <origin rpy="0 0 0" xyz="0 0 0.007"/>
+        <geometry>
+          <cylinder length="0.014" radius="0.030"/>
+        </geometry>
       </collision>
+    </link>
+    <joint name="${name}_anterior_gripper_joint" type="fixed">
+      <origin xyz="0 0 0.014" rpy="0 0 0"/>
+      <parent link="${name}_connector_link"/>
+      <child link="${name}_base_link"/>
+    </joint>
+    <!-- Base link -->
+    <link name="${name}_base_link">
       <inertial>
-        <origin xyz="0 0 ${adapter_h / 2}"/>
-        <mass value="0.15"/>
-        <inertia ixx="4.5e-5" ixy="0" ixz="0" iyy="4.5e-5" iyz="0" izz="8e-5"/>
+        <mass value="0.95"/>
+        <origin xyz="0 0 0"/>
+        <inertia ixx="1e-3" ixy="0" ixz="0" iyy="1e-3" iyz="0" izz="1e-3"/>
       </inertial>
-    </link>
-    <joint name="gripper_body_joint" type="fixed">
-      <parent link="gripper_adapter_link"/>
-      <child link="gripper_body_link"/>
-      <origin xyz="0 0 ${adapter_h}" rpy="0 0 0"/>
-    </joint>
-    <link name="gripper_body_link">
       <visual>
-        <origin xyz="0 0 ${body_h / 2}"/>
-        <geometry><box size="${body_x} ${body_y} ${body_h}"/></geometry>
-        <material name="wsg_grey"/>
+        <origin xyz="0 0 0" rpy="0 0 0"/>
+        <geometry>
+          <mesh filename="package://lwa4p_description/meshes/wsg_50/WSG50_BASE_110.stl" scale="1 1 1"/>
+        </geometry>
+        <material name="schunk_grey"/>
       </visual>
       <collision>
-        <origin xyz="0 0 ${body_h / 2}"/>
-        <geometry><box size="${body_x} ${body_y} ${body_h}"/></geometry>
+        <origin xyz="0 0 0" rpy="0 0 0"/>
+        <geometry>
+          <mesh filename="package://lwa4p_description/meshes/wsg_50/WSG50_BASE_110_collision.stl" scale="1.05 1.05 1.05"/>
+        </geometry>
       </collision>
-      <inertial>
-        <origin xyz="0 0 ${body_h / 2}"/>
-        <mass value="0.95"/>
-        <inertia ixx="6.1e-4" ixy="0" ixz="0" iyy="2.1e-3" iyz="0" izz="1.9e-3"/>
-      </inertial>
     </link>
-    <!-- the commanded joint: fingertip gap. Its link carries no geometry
-         (tiny inertial only so that Gazebo keeps the joint). -->
-    <joint name="gripper_joint" type="prismatic">
-      <parent link="gripper_body_link"/>
-      <child link="gripper_gap_link"/>
-      <origin xyz="0 0 ${body_h}" rpy="0 0 0"/>
+    <!-- Command joint for ros2_control -->
+    <joint name="${name}_joint" type="prismatic">
+      <parent link="${name}_base_link"/>
+      <child link="${name}_gap_link"/>
+      <origin xyz="0 0 0" rpy="0 0 0"/>
       <axis xyz="1 0 0"/>
-      <limit lower="0.0" upper="${gap_max}" effort="80" velocity="0.42"/>
+      <limit lower="0.0" upper="0.110" effort="80" velocity="0.42"/>
     </joint>
-    <link name="gripper_gap_link">
+    <link name="${name}_gap_link">
       <inertial>
         <mass value="0.01"/>
@@ -89,50 +68,121 @@
       </inertial>
     </link>
-    <!-- one finger = base jaw (on the housing top) + mounted finger.
-         Link origin: on the housing top, at the inner (gripping) face of the finger. -->
-    <xacro:macro name="finger" params="side sign">
-      <joint name="gripper_finger_${side}_joint" type="prismatic">
-        <parent link="gripper_body_link"/>
-        <child link="gripper_finger_${side}_link"/>
-        <origin xyz="0 0 ${body_h}" rpy="0 0 0"/>
-        <axis xyz="1 0 0"/>
-        <limit lower="${-gap_max}" upper="${gap_max}" effort="80" velocity="0.42"/>
-        <mimic joint="gripper_joint" multiplier="${sign * 0.5}" offset="0"/>
-      </joint>
-      <link name="gripper_finger_${side}_link">
-        <visual>
-          <origin xyz="${sign * (jaw_inset + jaw_w / 2)} 0 ${jaw_h / 2}"/>
-          <geometry><box size="${jaw_w} ${jaw_d} ${jaw_h}"/></geometry>
-          <material name="wsg_jaw"/>
-        </visual>
-        <visual>
-          <origin xyz="${sign * finger_t / 2} 0 ${jaw_h + finger_l / 2}"/>
-          <geometry><box size="${finger_t} ${finger_w} ${finger_l}"/></geometry>
-          <material name="wsg_black"/>
-        </visual>
-        <collision>
-          <origin xyz="${sign * (jaw_inset + jaw_w / 2)} 0 ${jaw_h / 2}"/>
-          <geometry><box size="${jaw_w} ${jaw_d} ${jaw_h}"/></geometry>
-        </collision>
-        <collision>
-          <origin xyz="${sign * finger_t / 2} 0 ${jaw_h + finger_l / 2}"/>
-          <geometry><box size="${finger_t} ${finger_w} ${finger_l}"/></geometry>
-        </collision>
-        <inertial>
-          <origin xyz="${sign * 0.012} 0 0.035"/>
-          <mass value="0.1"/>
-          <inertia ixx="5e-5" ixy="0" ixz="0" iyy="5.5e-5" iyz="0" izz="1.5e-5"/>
-        </inertial>
-      </link>
-    </xacro:macro>
-    <xacro:finger side="left" sign="-1"/>
-    <xacro:finger side="right" sign="1"/>
-    <!-- tool centre point: between the fingertips, 15 mm up from the tip -->
-    <joint name="gripper_tcp_joint" type="fixed">
-      <parent link="gripper_body_link"/>
-      <child link="gripper_tcp"/>
-      <origin xyz="0 0 ${body_h + jaw_h + finger_l - 0.015}" rpy="0 0 0"/>
+    <!-- Left finger base -->
+    <joint name="${name}_finger_left_joint" type="prismatic">
+      <parent link="${name}_base_link"/>
+      <child link="${name}_gripper_left"/>
+      <origin xyz="0 0 0" rpy="0 0 0"/>
+      <axis xyz="1 0 0"/>
+      <limit lower="-0.055" upper="0.055" effort="80" velocity="0.42"/>
+      <mimic joint="${name}_joint" multiplier="-0.5" offset="0"/>
     </joint>
-    <link name="gripper_tcp"/>
+    <link name="${name}_gripper_left">
+      <inertial>
+        <mass value="0.1"/>
+        <origin xyz="0 0 0"/>
+        <inertia ixx="1e-4" ixy="0" ixz="0" iyy="1e-4" iyz="0" izz="1e-4"/>
+      </inertial>
+      <visual>
+        <origin xyz="0 0 0" rpy="0 0 0"/>
+        <geometry>
+          <mesh filename="package://lwa4p_description/meshes/wsg_50/FINGERHOLD_WSG50.stl" scale="0.001 0.001 0.001"/>
+        </geometry>
+        <material name="schunk_grey"/>
+      </visual>
+      <collision>
+        <origin xyz="0 0 0" rpy="0 0 0"/>
+        <geometry>
+          <mesh filename="package://lwa4p_description/meshes/wsg_50/FINGERHOLD_WSG50.stl" scale="0.00105 0.00105 0.00105"/>
+        </geometry>
+      </collision>
+    </link>
+    <!-- Left finger tip -->
+    <joint name="${name}_guide_joint_finger_left" type="fixed">
+      <origin xyz="0 0 0.023" rpy="0 0 0"/>
+      <parent link="${name}_gripper_left"/>
+      <child link="${name}_finger_left_link"/>
+    </joint>
+    <link name="${name}_finger_left_link">
+      <inertial>
+        <mass value="0.1"/>
+        <origin xyz="0 0 0"/>
+        <inertia ixx="1e-4" ixy="0" ixz="0" iyy="1e-4" iyz="0" izz="1e-4"/>
+      </inertial>
+      <visual>
+        <origin xyz="0 0 0.001" rpy="0 0 0"/>
+        <geometry>
+          <mesh filename="package://lwa4p_description/meshes/wsg_50/WSG50_FINGER.stl" scale="0.001 0.001 0.001"/>
+        </geometry>
+        <material name="schunk_grey"/>
+      </visual>
+      <collision>
+        <origin xyz="-0.001 0 0.001" rpy="0 0 0"/>
+        <geometry>
+          <mesh filename="package://lwa4p_description/meshes/wsg_50/WSG50_FINGER.stl" scale="0.001 0.001 0.001"/>
+        </geometry>
+      </collision>
+    </link>
+    <!-- Right finger base -->
+    <joint name="${name}_finger_right_joint" type="prismatic">
+      <parent link="${name}_base_link"/>
+      <child link="${name}_gripper_right"/>
+      <origin xyz="0 0 0" rpy="0 0 3.14159"/>
+      <axis xyz="-1 0 0"/>
+      <limit lower="-0.055" upper="0.055" effort="80" velocity="0.42"/>
+      <mimic joint="${name}_joint" multiplier="0.5" offset="0"/>
+    </joint>
+    <link name="${name}_gripper_right">
+      <inertial>
+        <mass value="0.1"/>
+        <origin xyz="0 0 0"/>
+        <inertia ixx="1e-4" ixy="0" ixz="0" iyy="1e-4" iyz="0" izz="1e-4"/>
+      </inertial>
+      <visual>
+        <origin xyz="0 0 0" rpy="0 0 0"/>
+        <geometry>
+          <mesh filename="package://lwa4p_description/meshes/wsg_50/FINGERHOLD_WSG50.stl" scale="0.001 0.001 0.001"/>
+        </geometry>
+        <material name="schunk_grey"/>
+      </visual>
+      <collision>
+        <origin xyz="0 0 0" rpy="0 0 0"/>
+        <geometry>
+          <mesh filename="package://lwa4p_description/meshes/wsg_50/FINGERHOLD_WSG50.stl" scale="0.00105 0.00105 0.00105"/>
+        </geometry>
+      </collision>
+    </link>
+    <!-- Right finger tip -->
+    <joint name="${name}_guide_joint_finger_right" type="fixed">
+      <origin xyz="0 0 0.023" rpy="0 0 0"/>
+      <parent link="${name}_gripper_right"/>
+      <child link="${name}_finger_right_link"/>
+    </joint>
+    <link name="${name}_finger_right_link">
+      <inertial>
+        <mass value="0.1"/>
+        <origin xyz="0 0 0"/>
+        <inertia ixx="1e-4" ixy="0" ixz="0" iyy="1e-4" iyz="0" izz="1e-4"/>
+      </inertial>
+      <visual>
+        <origin xyz="0 0 0.001" rpy="0 0 0"/>
+        <geometry>
+          <mesh filename="package://lwa4p_description/meshes/wsg_50/WSG50_FINGER.stl" scale="0.001 0.001 0.001"/>
+        </geometry>
+        <material name="schunk_grey"/>
+      </visual>
+      <collision>
+        <origin xyz="-0.001 0 0.001" rpy="0 0 0"/>
+        <geometry>
+          <mesh filename="package://lwa4p_description/meshes/wsg_50/WSG50_FINGER.stl" scale="0.001 0.001 0.001"/>
+        </geometry>
+      </collision>
+    </link>
+    <!-- Tool center point -->
+    <joint name="${name}_tcp_joint" type="fixed">
+      <origin xyz="0 0 0.145" rpy="0 0 0"/>
+      <parent link="${name}_base_link"/>
+      <child link="${tool_point}"/>
+    </joint>
+    <link name="${tool_point}"/>
   </xacro:macro>
 </robot>
